File: TP-Final-DAC/tpfinal/tpfinal.kicad_pcb (KiCad board)
At the start: 2 copper layers, 108.1 x 81.5 mm, 17 parts, among them J1 220V, J2 1,5-30V 1,5A, SW2 SW_SPST, U1 LM317_TO-220

Commit message: Update
Parts:
- moved U1 4.98 mm to (131.0, 78.5)
- moved C2 4.98 mm to (136.1, 84.5)
- moved C4 4.20 mm to (118.5, 96.3)
- moved C3 4.20 mm to (125.6, 96.3)
- moved D2 3.91 mm to (146.1, 97.1)
- moved D4 1.06 mm to (115.8, 136.5)
- moved R1 0.08 mm to (135.9, 110.0)
Routing:
- net GND: track 0.00 -> 264.3 mm
- net +VDC: track 0.00 -> 153.6 mm
- net Net-(D3-A): track 0.00 -> 86.2 mm
- net Net-(J1-Pin_1): track 0.00 -> 43.5 mm
- net Net-(J1-Pin_2): track 71.7 -> 106.2 mm
- net Net-(D4-A): track 0.00 -> 15.9 mm
- net Net-(SW2-B): track 23.9 -> 29.0 mm
- net Net-(D1-+): track 60.0 -> 64.5 mm

Commit message: update
Parts:
- moved D4 0.64 mm to (115.8, 135.8)
Connections:
- TR1 pad 5: (no net) -> Net-(D1-Pad3)
Routing:
- net Net-(D1-Pad3): track 0.00 -> 91.3 mm
- net GND: track 264.3 -> 301.5 mm
- net Net-(F1-Pad2): track 45.3 -> 43.4 mm
- net Net-(D4-A): track 15.9 -> 15.3 mm
Changed lines of the file:
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@@
 			(layers "*.Cu" "*.Mask")
 			(remove_unused_layers no)
+			(net 6 "Net-(D1-Pad3)")
+			(pintype "passive")
 		)
 		(pad "6" thru_hole circle
@@
 		(embedded_fonts no)
 		(model "${KICAD9_3DMODEL_DIR}/Potentiometer_THT.3dshapes/Potentiometer_Piher_T-16H_Single_Horizontal.step"
+			(hide yes)
 			(offset
 				(xyz 0 0 0)
@@
 	(footprint "LED_THT:LED_D5.0mm_Horizontal_O3.81mm_Z9.0mm"
 		(layer "F.Cu")
-		(at 115.77 136.485)
+		(at 115.77 135.85)
 		(descr "LED, diameter 5.0mm, horizontal offset 3.81mm, z-position of LED center 9.0mm, 2 pins, generated by kicad-footprint-generator")
 		(tags "LED")
@@
 	)
 	(segment
+		(start 141.605 128.905)
+		(end 142.875 128.905)
+		(width 2)
+		(layer "B.Cu")
+		(net 1)
+	)
+	(segment
 		(start 143.51 97.79)
 		(end 143.51 113.665)
@@
 	)
 	(segment
+		(start 137.795 137.16)
+		(end 140.335 134.62)
+		(width 2)
+		(layer "B.Cu")
+		(net 1)
+	)
+	(segment
+		(start 143.51 113.665)
+		(end 143.51 127)
+		(width 2)
+		(layer "B.Cu")
+		(net 1)
+	)
+	(segment
 		(start 130.81 118.745)
 		(end 130.81 98.425)
@@
 	)
 	(segment
+		(start 113.905 96.28)
+		(end 116.349 96.28)
+		(width 2)
+		(layer "B.Cu")
+		(net 1)
+	)
+	(segment
 		(start 138.43 133.815)
 		(end 139.7 132.545)
@@
 	)
 	(segment
-		(start 130.81 98.425)
-		(end 128.665 96.28)
+		(start 139.7 128.905)
+		(end 137.795 127)
 		(width 2)
 		(layer "B.Cu")
@@
 	)
 	(segment
+		(start 137.795 128.905)
+		(end 137.795 127)
+		(width 2)
+		(layer "B.Cu")
+		(net 1)
+	)
+	(segment
 		(start 103.505 118.745)
 		(end 103.505 122.555)
@@
 	)
 	(segment
-		(start 113.905 96.28)
-		(end 116.349 96.28)
+		(start 105.42 125.095)
+		(end 105.42 124.46)
 		(width 2)
 		(layer "B.Cu")
@@
 	)
 	(segment
-		(start 105.42 125.095)
-		(end 105.42 124.46)
+		(start 140.97 133.985)
+		(end 141.355 133.985)
 		(width 2)
 		(layer "B.Cu")
@@
 	)
 	(segment
-		(start 140.97 133.985)
-		(end 141.355 133.985)
+		(start 115.77 137.36)
+		(end 116.461 138.051)
 		(width 2)
 		(layer "B.Cu")
@@
 	)
 	(segment
-		(start 137.795 128.905)
+		(start 137.795 127)
 		(end 137.795 123.825)
 		(width 2)
@@
 	)
 	(segment
+		(start 141.605 128.905)
+		(end 143.51 127)
+		(width 2)
+		(layer "B.Cu")
+		(net 1)
+	)
+	(segment
 		(start 143.51 129.54)
 		(end 143.51 131.83)
@@
 	)
 	(segment
+		(start 116.461 138.051)
+		(end 136.904 138.051)
+		(width 2)
+		(layer "B.Cu")
+		(net 1)
+	)
+	(segment
 		(start 112.395 106.68)
 		(end 112.395 97.79)
@@
 	)
 	(segment
-		(start 144.78 134.53)
-		(end 144.78 134.62)
+		(start 136.904 138.051)
+		(end 137.795 137.16)
 		(width 2)
 		(layer "B.Cu")
@@
 	)
 	(segment
-		(start 115.77 136.485)
-		(end 115.77 129.74)
+		(start 144.78 134.53)
+		(end 144.78 134.62)
 		(width 2)
 		(layer "B.Cu")
@@
 	(segment
 		(start 137.795 128.905)
-		(end 142.875 128.905)
+		(end 139.7 128.905)
 		(width 2)
 		(layer "B.Cu")
@@
 	)
 	(segment
+		(start 115.77 135.85)
+		(end 115.77 137.36)
+		(width 2)
+		(layer "B.Cu")
+		(net 1)
+	)
+	(segment
 		(start 147.955 132.545)
 		(end 147.955 132.715)
@@
 	)
 	(segment
-		(start 143.51 113.665)
+		(start 143.51 127)
 		(end 143.51 128.27)
 		(width 2)
@@
 	)
 	(segment
+		(start 139.7 128.905)
+		(end 141.605 128.905)
+		(width 2)
+		(layer "B.Cu")
+		(net 1)
+	)
+	(segment
 		(start 133.35 121.285)
 		(end 130.81 118.745)
@@
 	)
 	(segment
+		(start 130.81 98.425)
+		(end 128.665 96.28)
+		(width 2)
+		(layer "B.Cu")
+		(net 1)
+	)
+	(segment
 		(start 144.78 134.62)
 		(end 140.335 134.62)
@@
 	)
 	(segment
+		(start 115.77 129.74)
+		(end 115.77 135.85)
+		(width 2)
+		(layer "B.Cu")
+		(net 1)
+	)
+	(segment
 		(start 103.505 118.745)
 		(end 107.95 114.3)
@@
 	)
 	(segment
+		(start 137.795 137.16)
+		(end 137.795 132.545)
+		(width 2)
+		(layer "B.Cu")
+		(net 1)
+	)
+	(segment
 		(start 107.95 113.665)
 		(end 107.95 111.125)
@@
 	)
 	(segment
-		(start 118.31 136.485)
-		(end 118.31 120.555)
+		(start 190.5 71.12)
+		(end 188.595 71.12)
 		(width 2)
 		(layer "B.Cu")
-		(net 7)
+		(net 6)
 	)
 	(segment
-		(start 160.2 105.865)
-		(end 162.56 103.505)
+		(start 175.575 133.67)
+		(end 176.53 132.715)
 		(width 2)
 		(layer "B.Cu")
-		(net 8)
+		(net 6)
+	)
+	(segment
+		(start 192.405 80.01)
+		(end 192.405 73.025)
+		(width 2)
+		(layer "B.Cu")
+		(net 6)
+	)
+	(segment
+		(start 191.135 88.9)
+		(end 186.69 88.9)
+		(width 2)
+		(layer "B.Cu")
+		(net 6)
+	)
+	(segment
+		(start 176.53 109.855)
+		(end 179.705 106.68)
+		(width 2)
+		(layer "B.Cu")
+		(net 6)
+	)
+	(segment
+		(start 186.69 81.915)
+		(end 190.5 81.915)
+		(width 2)
+		(layer "B.Cu")
+		(net 6)
+	)
+	(segment
+		(start 185.42 83.185)
+		(end 186.69 81.915)
+		(width 2)
+		(layer "B.Cu")
+		(net 6)
 	)
 	(segment
-		(start 186.69 103.505)
-		(end 188.595 101.6)
+		(start 192.405 100.902684)
+		(end 192.405 90.17)
+		(width 2)
+		(layer "B.Cu")
+		(net 6)
+	)
+	(segment
+		(start 190.5 81.915)
+		(end 192.405 80.01)
+		(width 2)
+		(layer "B.Cu")
+		(net 6)
+	)
+	(segment
+		(start 179.705 106.68)
+		(end 186.627684 106.68)
+		(width 2)
+		(layer "B.Cu")
+		(net 6)
+	)
+	(segment
+		(start 171.185 133.67)
+		(end 175.575 133.67)
+		(width 2)
+		(layer "B.Cu")
+		(net 6)
+	)
+	(segment
+		(start 192.405 90.17)
+		(end 191.135 88.9)
+		(width 2)
+		(layer "B.Cu")
+		(net 6)
+	)
+	(segment
+		(start 185.42 87.63)
+		(end 185.42 83.185)
+		(width 2)
+		(layer "B.Cu")
+		(net 6)
+	)
+	(segment
+		(start 192.405 73.025)
+		(end 190.5 71.12)
+		(width 2)
+		(layer "B.Cu")
+		(net 6)
+	)
+	(segment
+		(start 176.53 132.715)
+		(end 176.53 109.855)
+		(width 2)
+		(layer "B.Cu")
+		(net 6)
+	)
+	(segment
+		(start 186.69 88.9)
+		(end 185.42 87.63)
+		(width 2)
+		(layer "B.Cu")
+		(net 6)
+	)
+	(segment
+		(start 186.627684 106.68)
+		(end 192.405 100.902684)
+		(width 2)
+		(layer "B.Cu")
+		(net 6)
+	)
+	(segment
+		(start 118.31 120.555)
+		(end 118.31 135.85)
+		(width 2)
+		(layer "B.Cu")
+		(net 7)
+	)
+	(segment
+		(start 160.2 105.865)
+		(end 166.37 99.695)
 		(width 2)
 		(layer "B.Cu")
@@
 	)
 	(segment
-		(start 162.56 103.505)
-		(end 186.69 103.505)
+		(start 187.325 99.695)
+		(end 188.595 98.425)
 		(width 2)
 		(layer "B.Cu")
@@
 	)
 	(segment
-		(start 188.595 101.6)
+		(start 188.595 98.425)
 		(end 188.595 91.12)
 		(width 2)
 		(layer "B.Cu")
+		(net 8)
+	)
+	(segment
+		(start 166.37 99.695)
+		(end 187.325 99.695)
+		(width 2)
+		(layer "B.Cu")
