File: TP-Final-DAC/TP-Final-DAC/tpfinal/tpfinal.kicad_pcb (KiCad board)
At the start: 2 copper layers, 108.1 x 81.5 mm, 17 parts, among them J1 220V, J2 1,5-30V 1,5A, SW2 SW_SPST, U1 LM317_TO-220

Commit message: Add files via upload
Parts:
- D1: footprint Package_SO:TSSOP-4_4.4x5mm_P4mm -> Diode_THT:Diode_Bridge_16.7x16.7x6.3mm_P10.8mm
- moved D1 44.3 mm to (136.5, 99.1)
- moved C4 32.0 mm to (114.3, 104.2), turned to 90 degrees
- moved R2 31.1 mm to (120.0, 114.9)
- moved J2 30.8 mm to (110.5, 120.0), turned to 180 degrees
- moved D3 26.1 mm to (125.7, 104.1)
- moved C1 22.9 mm to (142.2, 87.6), turned to 180 degrees
- moved F1 18.8 mm to (149.7, 120.7), turned to 180 degrees
- moved D2 18.6 mm to (141.6, 77.5)
- moved C3 15.6 mm to (125.6, 85.7)
- moved C2 11.3 mm to (135.9, 77.4), turned to 180 degrees
- moved R1 6.49 mm to (128.9, 78.1), turned to 180 degrees
- moved TR1 4.36 mm to (188.4, 108.4)
- moved D4 2.33 mm to (114.9, 133.9)
- moved SW2 2.32 mm to (147.2, 133.7)
- moved U1 2.12 mm to (130.8, 70.2), turned to 0 degrees
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Connections:
- SW2 pad 1: Net-(J1-Pin_2) -> Net-(SW2-B)
- SW2 pad 2: Net-(SW2-B) -> Net-(J1-Pin_2)
- TR1 pad 5: (no net) -> Net-(D1-Pad3)
Routing:
- net GND: track 0.00 -> 348.6 mm
- net +VDC: track 0.00 -> 197.6 mm
- net Net-(J1-Pin_2): track 0.00 -> 156.6 mm
- net Net-(D3-A): track 0.00 -> 108.7 mm
- net Net-(F1-Pad2): track 0.00 -> 102.5 mm
- net Net-(D1-Pad4): track 0.00 -> 67.1 mm
- net Net-(D1-Pad3): track 0.00 -> 64.3 mm
- net Net-(SW2-B): track 0.00 -> 61.9 mm
- net Net-(J1-Pin_1): track 0.00 -> 56.4 mm
- net Net-(D1-+): track 0.00 -> 39.4 mm
- net Net-(D4-A): track 0.00 -> 10.7 mm
