File: TP-Final-DAC/TP-Final-DAC/tpfinal/tpfinal.kicad_sch (KiCad schematic)
At the start: 17 parts, among them J1 220V, J2 1,5-30V 1,5A, SW2 SW_SPST, U1 LM317_TO-220

Commit message: Add files via upload
Parts:
- D1: footprint Package_SO:TSSOP-4_4.4x5mm_P4mm -> Diode_THT:Diode_Bridge_16.7x16.7x6.3mm_P10.8mm
Connections:
- net at J1.2 (Pin_2): now also SW2.2 (A); no longer SW2.1 (A)
- net at F1.1: now also SW2.1 (B); no longer SW2.2 (B)
Changed lines of the file:
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@@
 			)
-		)
-		(pin "1"
 		)
 		(pin "2"
+		)
+		(pin "1"
 		)
 		(instances
@@
 			)
 		)
-		(property "Footprint" "Package_SO:TSSOP-4_4.4x5mm_P4mm"
+		(property "Footprint" "Diode_THT:Diode_Bridge_16.7x16.7x6.3mm_P10.8mm"
 			(at 102.87 99.06 0)
 			(effects
