File: tpfinal.kicad_sch (KiCad schematic)
At the start: 17 parts, among them J1 220V, J2 1,5-30V 1,5A, SW2 SW_SPST, U1 LM317_TO-220

Commit message: Update
Connections:
- net at D1.3: now also TR1.5; no longer TR1.3
Other:
- company: (none) -> Bolanho Alejo Eloy
- title: (none) -> SCH Trabajo Final Integrador
Changed lines of the file:
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@@
 	(generator_version "9.0")
 	(paper "A4")
+	(title_block
+		(title "SCH Trabajo Final Integrador")
+		(date "2025-10-23")
+		(rev "1.0")
+		(company "Bolanho Alejo Eloy")
+		(comment 1 "416154")
+		(comment 2 "1R5")
+	)
 	(junction
 		(at 125.73 76.2)
@@
 		(pin "4"
 		)
-		(pin "3"
+		(pin "5"
 		)
 		(instances
